File: hardware/dielectric-module/MS-DIEL-CTRL.kicad_pcb (KiCad board)
At the start: 4 copper layers, 130 x 100 mm, 60 parts, among them J1 24V_IN, J2 CAN, J3 FLUSH_SOL, J4 PUMP_CHILL_DEION, J5 ANALOG_SENSORS, J6 TEMP_1WIRE, J7 FLOW_FLOATS, J8 USB-C, Q1 AO3400, Q2 AO3400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

Commit message: hw(dielectric): schematic-first (option A) — linked schematic + PCB from one model
generate.py builds MS-DIEL-CTRL.kicad_sch (source of truth) and MS-DIEL-CTRL.kicad_pcb
from one PARTS+NETS model. Footprints carry the same UUID as their schematic symbol
(linkage proven: footprint path == symbol uuid), so Update-PCB-from-Schematic/ERC work.
ICs wired by real library pin names (authoritative pinouts: MCP2518FD SCK=10/SDI=11/
SDO=12/CS=13, etc.), ESP32 by GPIO name. Schematic loads in KiCad 10, ERC = 36 benign
warnings (unused GPIOs, PWR_FLAG nags, symbol-cache notes), netlist correct.

Notable [REVIEW] changes from the scaffold: buck AP3402, reverse-FET AO3401A, USB-C
replaced by a 6-pin USB/UART programming header (avoids pad-name mismatch). Supersedes
the PCB-only generate_board.py (removed). PSU board remains the earlier scaffold.
Parts:
- removed R5: 5k1_CC1, R_0805_2012Metric
- removed R6: 5k1_CC2, R_0805_2012Metric
- C3: value 1uF_EN -> 1uF
- C4: value 100nF_IO0 -> 100nF
- D1: value fly1 -> fly
- D2: value fly2 -> fly
- D3: value fly3 -> fly
- D5: value SMBJ24A_TVS -> SMBJ24A
- D6: value B340_cat -> B340
- J8: value USB-C -> PROG_USB; footprint USB_C_Receptacle_Amphenol_12401548E4-2A -> PinHeader_1x06_P2.54mm_Vertical
- Q1, Q2, Q3, Q4, Q5, Q6: value AO3400 -> AO3400A
- Q7: value DMP_revprot -> AO3401A
- R1: value 10k_EN -> 10k
- R2: value 10k_IO0 -> 10k
- R3: value 120R_term -> 120R
- R4: value 4k7_1wire_pullup -> 4k7
- Rc1, Rc2: value div_cond -> div
- Rl1, Rl2: value div_level -> div
- Rp1, Rp2: value div_press -> div
- U3: value TJA1051T/3 -> TJA1051T-3
- U4: value MP2316_buck -> AP3402
- moved D5 4.00 mm to (18.0, 20.0)
Connections:
- D5 pad 1: GND -> +24V
- D5 pad 2: +24V -> GND
- D6 pad 2: SW5 -> SW
- J2 pad 3: CAN_GND -> GND
- J3 pad 4: J3_24a -> +24V
- J3 pad 5: J3_24b -> +24V
- J4 pad 4: J4_x -> GND
- J4 pad 5: J4_y -> GND
- L1 pad 1: SW5 -> SW
- Q7 pad 1: (no net) -> GND
- Q7 pad 2: GND -> 24V_RAW
- R2 pad 2: IO0R -> +3V3
- R7 pad 2: FB5 -> FB
- R8 pad 1: FB5 -> FB
- Rc2 pad 2: COND_GND -> GND
- Rl2 pad 2: LEVEL_GND -> GND
- Rp2 pad 2: PRESS_GND -> GND
- U2 pad 1: OSC1 -> MCP_TXCAN
- U2 pad 10: MCP_TXCAN -> SPI_SCK
- U2 pad 11: MCP_RXCAN -> SPI_MOSI
- U2 pad 12: (no net) -> SPI_MISO
- U2 pad 13: +3V3 -> MCP_CS
- U2 pad 14: GND -> +3V3
- U2 pad 2: OSC2 -> MCP_RXCAN
- U2 pad 3: MCP_INT -> (no net)
- U2 pad 4: SPI_SCK -> MCP_INT
- U2 pad 5: SPI_MOSI -> OSC2
- U2 pad 6: SPI_MISO -> OSC1
- U2 pad 7: MCP_CS -> GND
- U4 pad 1: SW5 -> +24V
- U4 pad 2: +24V -> GND
- U4 pad 3: GND -> SW
- U4 pad 4: FB5 -> +24V
- U4 pad 6: (no net) -> FB

Commit message: hw(dielectric): human-readable schematic engine (power glyphs, stubbed labels, blocks, NC, PWR_FLAG, title); add missing MCP2518FD crystal; ERC 0 errors
Parts:
- added C11: 18pF, C_0805_2012Metric, F.Cu at (108.0, 44.0)
- added C12: 18pF, C_0805_2012Metric, F.Cu at (116.0, 44.0)
- added Y1: 40MHz, Crystal_SMD_3215-2Pin_3.2x1.5mm, F.Cu at (112.0, 40.0)

Commit message: hw(dielectric): assign real values to FB divider, sensor dividers, solenoid flyback diodes
Parts:
- D1, D2, D3: value fly -> 1N4007
- R7: value FB_top -> 75k
- R8: value FB_bot -> 10k
- Rc1, Rl1, Rp1: value div -> 10k
- Rc2, Rl2, Rp2: value div -> 20k
